File: schematic/at28c64b-15pu-programmer.sch (KiCad schematic (older format))
At the start: 8 parts, among them U1 ARDUINO NANO, U2 AT28C64B-15PU, U3 74HC595, U4 74HC595

Commit message: Tidy up the schematic a bit
Connections:
- net Arduino5V: now also C8.1
- net GND: now also C8.2
Other:
- moved on the sheet: C2, C3, C8, U3, U4
