File: schematic/eeprom-programmer.sch (KiCad schematic (older format))
At the start: 8 parts, among them U1 ARDUINO NANO, U2 AT28C64B-15PU, U3 74HC595, U4 74HC595

Commit message: Readd Arduino and EEPROM symbols
Parts:
- removed C2, C3, C4, C8: .1uF, symbol Device:C
- removed U1: ARDUINO NANO, ARDUINO_A000005, symbol at28c64b-15pu-programmer-rescue:A000005-Arduino
- removed U2: AT28C64B-15PU, DIP254P1524X482-28, symbol at28c64b-15pu-programmer-rescue:AT28C64B-15PU-eeprom
- removed U3, U4: 74HC595, symbol 74xx:74HC595
- added A1: Arduino_Nano_v3.x, Module:Arduino_Nano, symbol eeprom-programmer:Arduino_Nano_v3.x
- added C1, C2, C3, C4: .1uF, symbol eeprom-programmer:C
- added IC?: AT28C64B-15PU, DIP1556W56P254L3702H483Q28N, symbol eeprom-programmer:AT28C64B-15PU
- added U1, U2: 74HC595, symbol eeprom-programmer:74HC595
Connections:
- net labels added: address0, address1, address10, address11, address12, address2, address3, address4, address5, address6, address7, address8, address9
- net labels removed: addr0, addr1, addr10, addr11, addr12, addr2, addr3, addr4, addr5, addr6, addr7, addr8, addr9
- wire segments 72 -> 27
Other:
- note removed: "1"

Commit message: Remove excess wires
Parts:
- gave numbers to parts that had none: 1
Connections:
- wire segments 27 -> 13
Changed lines of the file:
@@
 Text GLabel 9150 3400 2    50   Input ~ 0
 eeNotWriteEnable
-Wire Wire Line
-	2000 2600 1800 2600
-Text GLabel 1800 2600 0    50   Input ~ 0
+Text GLabel 2000 2600 0    50   Input ~ 0
 srSerialData
-Text GLabel 1800 2800 0    50   Input ~ 0
+Text GLabel 2000 2800 0    50   Input ~ 0
 srSerialClock
-Text GLabel 1800 4900 0    50   Input ~ 0
+Text GLabel 2000 4900 0    50   Input ~ 0
 srSerialClock
-Text GLabel 1800 2900 0    50   Input ~ 0
+Text GLabel 2000 2900 0    50   Input ~ 0
 srNotResetAll
-Wire Wire Line
-	2000 5000 1800 5000
-Text GLabel 1800 5000 0    50   Input ~ 0
+Text GLabel 2000 5000 0    50   Input ~ 0
 srNotResetAll
-Wire Wire Line
-	2000 3100 1800 3100
-Text GLabel 1800 3100 0    50   Input ~ 0
+Text GLabel 2000 3100 0    50   Input ~ 0
 srReadClock
-Wire Wire Line
-	2000 5200 1800 5200
-Text GLabel 1800 5200 0    50   Input ~ 0
+Text GLabel 2000 5200 0    50   Input ~ 0
 srReadClock
-Wire Wire Line
-	2000 3200 1800 3200
-Text GLabel 1800 3200 0    50   Input ~ 0
+Text GLabel 2000 3200 0    50   Input ~ 0
 srNotOutputEnable
-Wire Wire Line
-	2000 5300 1800 5300
-Text GLabel 1800 5300 0    50   Input ~ 0
+Text GLabel 2000 5300 0    50   Input ~ 0
 srNotOutputEnable
-Wire Wire Line
-	1800 2800 2000 2800
-Wire Wire Line
-	1800 4900 2000 4900
-Wire Wire Line
-	2000 2900 1800 2900
 Text GLabel 2400 2000 0    50   Input ~ 0
 Arduino5V
@@
 Text GLabel 5750 2550 1    50   Output ~ 0
 Arduino5V
-Text GLabel 6200 4350 2    50   Output ~ 0
+Text GLabel 6050 4350 2    50   Output ~ 0
 srSerialData
-Text GLabel 6200 4250 2    50   Output ~ 0
+Text GLabel 6050 4250 2    50   Output ~ 0
 srSerialClock
 Text Notes 7350 7500 0    50   ~ 0
@@
 Wire Wire Line
 	2800 3500 2800 4000
-Text GLabel 6200 4150 2    50   Output ~ 0
+Text GLabel 6050 4150 2    50   Output ~ 0
 srNotOutputEnable
-Text GLabel 6200 4050 2    50   Output ~ 0
+Text GLabel 6050 4050 2    50   Output ~ 0
 srReadClock
-Text GLabel 6200 3950 2    50   Output ~ 0
+Text GLabel 6050 3950 2    50   Output ~ 0
 srNotResetAll
 Text GLabel 5050 4350 0    50   Output ~ 0
@@
 $EndComp
 NoConn ~ 6050 3750
-Wire Wire Line
-	6050 3950 6200 3950
-Wire Wire Line
-	6050 4050 6200 4050
-Wire Wire Line
-	6050 4150 6200 4150
-Wire Wire Line
-	6050 4250 6200 4250
-Wire Wire Line
-	6050 4350 6200 4350
 NoConn ~ 6050 4450
 $Comp
-L eeprom-programmer:AT28C64B-15PU IC?
+L eeprom-programmer:AT28C64B-15PU IC1
 U 1 1 5CB76AFF
 P 8050 3300
-F 0 "IC?" H 8600 3565 50  0000 C CNN
+F 0 "IC1" H 8600 3565 50  0000 C CNN
 F 1 "AT28C64B-15PU" H 8600 3474 50  0000 C CNN
 F 2 "DIP1556W56P254L3702H483Q28N" H 9000 3400 50  0001 L CNN

Commit message: Add busses
Parts:
- renumbered C4 to C1, C1 to C2, C2 to C3, C3 to C4
Connections:
- net labels added: addr00, addr01, addr02, addr03, addr04, addr05, addr06, addr07, addr08, addr09, addr10, addr11, addr12
- net labels removed: address0, address1, address10, address11, address12, address2, address3, address4, address5, address6, address7, address8, address9
- wire segments 13 -> 55
