File: schematic/eeprom-programmer.sch (KiCad schematic (older format))
At the start: 8 parts, among them IC1 AT28C64B-15PU, U1 74HC595, U2 74HC595

Commit message: Updated schematic to handle up to 32Kx8 eeproms with no rewiring
Parts:
- removed C1, C2, C3, C4: .1uF, Capacitor_THT:C_Disc_D5.0mm_W2.5mm_P5.00mm, symbol eeprom-programmer:C
- removed IC1: AT28C64B-15PU, Package_DIP:DIP-28_W15.24mm_Socket, symbol eeprom-programmer:AT28C64B-15PU
- removed U1, U2: 74HC595, Package_DIP:DIP-16_W7.62mm_Socket, symbol eeprom-programmer:74HC595
- added IC1: AT28C256-15PU, DIP1556W56P254L3702H483Q28N, symbol eeprom-programmer:AT28C256-15PU
- added U1, U2: 74LS595, symbol eeprom-programmer:74LS595
Connections:
- net labels added: addr13, addr14
- no-connect marks 14 -> 12

Commit message: Update PCB layout to handle up to 32kx8 eeproms
Parts:
- added C1, C2, C3: .1uf, eeprom-programmer:C_Disc_D5.0mm_W2.5mm_P5.00mm, symbol Device:C
- A1: footprint Module:Arduino_Nano -> eeprom-programmer:Arduino_Nano
- IC1: footprint DIP1556W56P254L3702H483Q28N -> eeprom-programmer:DIP254P1524X482-28
- U1, U2: footprint (none) -> eeprom-programmer:DIP254P762X508-16
Connections:
- wire segments 55 -> 58
Changed lines of the file:
@@
 EESchema Schematic File Version 4
-EELAYER 29 0
+EELAYER 30 0
 EELAYER END
 $Descr A 11000 8500
@@
 Connection ~ 6300 5050
 Wire Wire Line
-	7850 2300 7850 2700
-Wire Wire Line
 	3400 2300 3400 2700
 $Comp
@@
 F 0 "A1" H 3200 2611 50  0000 C CNN
 F 1 "Arduino_Nano_v3.x" H 3200 2520 50  0000 C CNN
-F 2 "Module:Arduino_Nano" H 3350 2750 50  0001 L CNN
+F 2 "eeprom-programmer:Arduino_Nano" H 3350 2750 50  0001 L CNN
 F 3 "http://www.mouser.com/pdfdocs/Gravitech_Arduino_Nano3_0.pdf" H 3200 2700 50  0001 C CNN
 	1    3200 3700
@@
 $EndComp
 Wire Wire Line
-	5500 1750 5500 2150
-Wire Wire Line
-	5500 3950 5500 4350
+	5500 1750 5500 1850
+Wire Wire Line
+	5500 3950 5500 4050
 $Comp
 L eeprom-programmer:74LS595 U1
@@
 F 0 "U1" H 5500 3531 50  0000 C CNN
 F 1 "74LS595" H 5500 3440 50  0000 C CNN
-F 2 "" H 5500 2750 50  0001 C CNN
+F 2 "eeprom-programmer:DIP254P762X508-16" H 5500 2750 50  0001 C CNN
 F 3 "http://www.ti.com/lit/gpn/sn74ls595" H 5500 2750 50  0001 C CNN
 	1    5500 2750
@@
 F 0 "U2" H 5500 5731 50  0000 C CNN
 F 1 "74LS595" H 5500 5640 50  0000 C CNN
-F 2 "" H 5500 4950 50  0001 C CNN
+F 2 "eeprom-programmer:DIP254P762X508-16" H 5500 4950 50  0001 C CNN
 F 3 "http://www.ti.com/lit/gpn/sn74ls595" H 5500 4950 50  0001 C CNN
 	1    5500 4950
@@
 F 0 "IC1" H 7850 3481 50  0000 C CNN
 F 1 "AT28C256-15PU" H 7850 3390 50  0000 C CNN
-F 2 "DIP1556W56P254L3702H483Q28N" H 6800 4300 50  0001 L CNN
+F 2 "eeprom-programmer:DIP254P1524X482-28" H 6800 4300 50  0001 L CNN
 F 3 "https://componentsearchengine.com/Datasheets/1/AT28C64B-15PU.pdf" H 6800 4200 50  0001 L CNN
 F 4 "AT28C256-15PU, Parallel EEPROM Memory 256kbit, Parallel, 150ns 4.5  5.5 V, 28-Pin PDIP" H 6800 4100 50  0001 L CNN "Description"
@@
 	8700 4400 8800 4500
 $Comp
-L power:GND #PWR?
+L power:GND #PWR0101
 U 1 1 5DEC1A08
 P 3300 5100
-F 0 "#PWR?" H 3300 4850 50  0001 C CNN
+F 0 "#PWR0101" H 3300 4850 50  0001 C CNN
 F 1 "GND" V 3305 4972 50  0000 R CNN
 F 2 "" H 3300 5100 50  0001 C CNN
@@
 $EndComp
 $Comp
-L power:GND #PWR?
+L power:GND #PWR0102
 U 1 1 5DEC3279
 P 5500 5650
-F 0 "#PWR?" H 5500 5400 50  0001 C CNN
+F 0 "#PWR0102" H 5500 5400 50  0001 C CNN
 F 1 "GND" V 5505 5522 50  0000 R CNN
 F 2 "" H 5500 5650 50  0001 C CNN
@@
 $EndComp
 $Comp
-L power:GND #PWR?
+L power:GND #PWR0103
 U 1 1 5DEC4AEA
 P 5500 3450
-F 0 "#PWR?" H 5500 3200 50  0001 C CNN
+F 0 "#PWR0103" H 5500 3200 50  0001 C CNN
 F 1 "GND" V 5505 3322 50  0000 R CNN
 F 2 "" H 5500 3450 50  0001 C CNN
@@
 $EndComp
 $Comp
-L power:GND #PWR?
+L power:GND #PWR0104
 U 1 1 5DEC63E4
 P 7850 4700
-F 0 "#PWR?" H 7850 4450 50  0001 C CNN
+F 0 "#PWR0104" H 7850 4450 50  0001 C CNN
 F 1 "GND" V 7855 4572 50  0000 R CNN
 F 2 "" H 7850 4700 50  0001 C CNN
@@
 $EndComp
 $Comp
-L power:GND #PWR?
+L power:GND #PWR0105
 U 1 1 5DEC7D0B
 P 5900 5250
-F 0 "#PWR?" H 5900 5000 50  0001 C CNN
+F 0 "#PWR0105" H 5900 5000 50  0001 C CNN
 F 1 "GND" V 5905 5122 50  0000 R CNN
 F 2 "" H 5900 5250 50  0001 C CNN
@@
 $EndComp
 $Comp
-L power:GND #PWR?
+L power:GND #PWR0106
 U 1 1 5DEC957C
 P 5900 5450
-F 0 "#PWR?" H 5900 5200 50  0001 C CNN
+F 0 "#PWR0106" H 5900 5200 50  0001 C CNN
 F 1 "GND" V 5905 5322 50  0000 R CNN
 F 2 "" H 5900 5450 50  0001 C CNN
@@
 	0    -1   -1   0
 $EndComp
+$Comp
+L Device:C C1
+U 1 1 5E0AC806
+P 5650 1850
+F 0 "C1" V 5398 1850 50  0000 C CNN
+F 1 ".1uf" V 5489 1850 50  0000 C CNN
+F 2 "eeprom-programmer:C_Disc_D5.0mm_W2.5mm_P5.00mm" H 5688 1700 50  0001 C CNN
+F 3 "~" H 5650 1850 50  0001 C CNN
+	1    5650 1850
+	0    1    1    0
+$EndComp
+Connection ~ 5500 1850
+Wire Wire Line
+	5500 1850 5500 2150
+$Comp
+L Device:C C2
+U 1 1 5E0AD397
+P 5650 4050
+F 0 "C2" V 5398 4050 50  0000 C CNN
+F 1 ".1uf" V 5489 4050 50  0000 C CNN
+F 2 "eeprom-programmer:C_Disc_D5.0mm_W2.5mm_P5.00mm" H 5688 3900 50  0001 C CNN
+F 3 "~" H 5650 4050 50  0001 C CNN
+	1    5650 4050
+	0    1    1    0
+$EndComp
+Connection ~ 5500 4050
+Wire Wire Line
+	5500 4050 5500 4350
+$Comp
+L Device:C C3
+U 1 1 5E0ADC8B
+P 8000 2400
+F 0 "C3" V 7748 2400 50  0000 C CNN
+F 1 ".1uf" V 7839 2400 50  0000 C CNN
+F 2 "eeprom-programmer:C_Disc_D5.0mm_W2.5mm_P5.00mm" H 8038 2250 50  0001 C CNN
+F 3 "~" H 8000 2400 50  0001 C CNN
+	1    8000 2400
+	0    1    1    0
+$EndComp
+$Comp
+L eeprom-programmer:GND #PWR0107
+U 1 1 5E0AE377
+P 5800 1850
+F 0 "#PWR0107" H 5800 1600 50  0001 C CNN
+F 1 "GND" V 5805 1722 50  0000 R CNN
+F 2 "" H 5800 1850 50  0001 C CNN
+F 3 "" H 5800 1850 50  0001 C CNN
+	1    5800 1850
+	0    -1   -1   0
+$EndComp
+$Comp
+L eeprom-programmer:GND #PWR0108
+U 1 1 5E0AED53
+P 5800 4050
+F 0 "#PWR0108" H 5800 3800 50  0001 C CNN
+F 1 "GND" V 5805 3922 50  0000 R CNN
+F 2 "" H 5800 4050 50  0001 C CNN
+F 3 "" H 5800 4050 50  0001 C CNN
+	1    5800 4050
+	0    -1   -1   0
+$EndComp
+Wire Wire Line
+	7850 2300 7850 2400
+Connection ~ 7850 2400
+Wire Wire Line
+	7850 2400 7850 2700
+$Comp
+L eeprom-programmer:GND #PWR0109
+U 1 1 5E0B56EB
+P 8150 2400
+F 0 "#PWR0109" H 8150 2150 50  0001 C CNN
+F 1 "GND" V 8155 2272 50  0000 R CNN
+F 2 "" H 8150 2400 50  0001 C CNN
+F 3 "" H 8150 2400 50  0001 C CNN
+	1    8150 2400
+	0    -1   -1   0
+$EndComp
